Commit message: switched out lidar for simple_wamv

File: all_seaing_ros2/urdf/simple_wamv/simple_component_config.xacro (robot description, xacro)
@@ -11,5 +11,5 @@
       <xacro:wamv_imu name="imu_wamv" x="0.3" y="-0.2" z="1.3" R="0.0" P="0.0" Y="0.0" />
     <!-- === lidar === -->
-      <xacro:lidar name="lidar_wamv" type="16_beam" x="0.7" y="0.0" z="1.8" R="0.0" P="${radians(8)}" Y="0.0" post_Y="0.0" />
+      <xacro:lidar name="lidar_wamv" type="32_beam" x="0.7" y="0.0" z="1.8" R="0.0" P="${radians(8)}" Y="0.0" post_Y="0.0" />
     <!-- === wamv_ball_shooter === -->
       <xacro:wamv_ball_shooter name="ball_shooter" x="0.55" y="-0.3" z="1.3" pitch="${radians(-20)}" yaw="0.0" />

File: all_seaing_ros2/urdf/simple_wamv/simple_thruster_config.xacro (robot description, xacro)
@@ -5,8 +5,6 @@
       <xacro:engine prefix="left" position="-2.373776 1.027135 0.318237" orientation="0.0 0.0 0.0" />
       <xacro:engine prefix="right" position="-2.373776 -1.027135 0.318237" orientation="0.0 0.0 0.0" />
-      <xacro:engine prefix="middle" position="0 0 0.318237" orientation="0.0 0.0 0.0" />
       <xacro:include filename="$(find wamv_gazebo)/urdf/thruster_layouts/wamv_gazebo_thruster_config.xacro" />
         <xacro:wamv_gazebo_thruster_config name="left" />
         <xacro:wamv_gazebo_thruster_config name="right" />
-        <xacro:wamv_gazebo_thruster_config name="middle" />
 </robot>

File: all_seaing_ros2/urdf/simple_wamv/wamv_target.urdf (robot description, URDF)
Before this commit: robot WAM-V, 30 links, 29 joints
Links:
- removed link wamv/middle_engine_link
- removed link wamv/middle_propeller_link
Joints:
- removed joint wamv/middle_chassis_engine_joint
- removed joint wamv/middle_engine_propeller_joint
