Commit message: fixed wamv urdf, fixed xdrive sim yaml file

File: all_seaing_ros2/urdf/xdrive_wamv/wamv_target.urdf (robot description, URDF)
Before this commit: robot WAM-V, 12 links, 11 joints
Links:
- added link wamv/gps_wamv_link, mass 1; collision cylinder length=0.05 radius=0.015; collision cylinder length=0.1 radius=0.15
- added link wamv/imu_wamv_link, mass 0.1; collision box size=0.05 0.025 0.005; visual box size=0.05 0.025 0.005
Joints:
- added joint wamv/gps_wamv_joint: type revolute, parent wamv/base_link, child wamv/gps_wamv_link, origin xyz=-0.65 0.0 1.3 rpy=0.0 0.0 0.0, axis 0 0 1, limit lower=0.0 upper=0 effort=1000.0 velocity=0
- added joint wamv/imu_wamv_joint: type revolute, parent wamv/base_link, child wamv/imu_wamv_link, origin xyz=-0.65 0.0 1.3 rpy=0.0 0.0 0.0, axis 0 0 1, limit lower=0.0 upper=0 effort=1000.0 velocity=0
- joint wamv/back_left_chassis_engine_joint: origin xyz=-2.25 1 0.318237 rpy=0.0 0.0 0.7854 -> xyz=-2.4 1 0 rpy=0.0 0.0 0.7854
- joint wamv/back_right_chassis_engine_joint: origin xyz=-2.25 -1 0.318237 rpy=0.0 0.0 -0.7854 -> xyz=-2.4 -1 0 rpy=0.0 0.0 -0.7854
- joint wamv/front_left_chassis_engine_joint: origin xyz=1.25 1 0.318237 rpy=0.0 0.0 -0.7854 -> xyz=1.1 1 0 rpy=0.0 0.0 -0.7854
- joint wamv/front_right_chassis_engine_joint: origin xyz=1.25 -1 0.318237 rpy=0.0 0.0 0.7854 -> xyz=1.1 -1 0 rpy=0.0 0.0 0.7854

File: all_seaing_ros2/urdf/xdrive_wamv/xdrive_component_config.xacro (robot description, xacro)
@@ -2,4 +2,8 @@
 <robot xmlns:xacro="http://ros.org/wiki/xacro" name="wam-v-components">
   <xacro:macro name="yaml_components">
+    <!-- === wamv_imu === -->
+      <xacro:wamv_imu name="imu_wamv" x="-0.65" y="0.0" z="1.3" R="0.0" P="0.0" Y="0.0" />
+    <!-- === wamv_gps === -->
+      <xacro:wamv_gps name="gps_wamv" x="-0.65" y="0.0" z="1.3" R="0.0" P="0.0" Y="0.0" />
   </xacro:macro>
 </robot>

File: all_seaing_ros2/urdf/xdrive_wamv/xdrive_thruster_config.xacro (robot description, xacro)
@@ -3,8 +3,8 @@
   <xacro:include filename="$(find wamv_description)/urdf/thrusters/engine.xacro" />
     <!-- === engine === -->
-      <xacro:engine prefix="front_left" position="1.25 1 0.318237" orientation="0.0 0.0 -0.7854" />
-      <xacro:engine prefix="front_right" position="1.25 -1 0.318237" orientation="0.0 0.0 0.7854" />
-      <xacro:engine prefix="back_left" position="-2.25 1 0.318237" orientation="0.0 0.0 0.7854" />
-      <xacro:engine prefix="back_right" position="-2.25 -1 0.318237" orientation="0.0 0.0 -0.7854" />
+      <xacro:engine prefix="front_left" position="1.1 1 0" orientation="0.0 0.0 -0.7854" />
+      <xacro:engine prefix="front_right" position="1.1 -1 0" orientation="0.0 0.0 0.7854" />
+      <xacro:engine prefix="back_left" position="-2.4 1 0" orientation="0.0 0.0 0.7854" />
+      <xacro:engine prefix="back_right" position="-2.4 -1 0" orientation="0.0 0.0 -0.7854" />
       <xacro:include filename="$(find wamv_gazebo)/urdf/thruster_layouts/wamv_gazebo_thruster_config.xacro" />
         <xacro:wamv_gazebo_thruster_config name="front_left" />

Commit message: converted follow the path to xdrive, added cameras and lidar to xdrive urdf

File: all_seaing_ros2/urdf/xdrive_wamv/wamv_target.urdf (robot description, URDF)
Before this commit: robot WAM-V, 14 links, 13 joints
Links:
- added link wamv/far_left_camera_link, mass 0.3; collision box size=0.036 0.03 0.03; collision cylinder length=0.042 radius=0.015
- added link wamv/far_left_camera_link_optical
- added link wamv/far_left_camera_post_arm_link, mass 0.1; collision cylinder length=0.065 radius=0.008; visual mesh filename=package://vrx_gazebo/models/sensor_post/mesh/sensor_post_ar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
- added link wamv/far_left_camera_post_link, mass 0.15885000000000002; collision cylinder length=0.17650000000000002 radius=0.0076; visual cylinder length=0.17650000000000002 radius=0.0076
- added link wamv/front_left_camera_link, mass 0.3; collision box size=0.036 0.03 0.03; collision cylinder length=0.042 radius=0.015
- added link wamv/front_left_camera_link_optical
- added link wamv/front_left_camera_post_arm_link, mass 0.1; collision cylinder length=0.065 radius=0.008; visual mesh filename=package://vrx_gazebo/models/sensor_post/mesh/sensor_post_ar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
- added link wamv/front_left_camera_post_link, mass 0.15885000000000002; collision cylinder length=0.17650000000000002 radius=0.0076; visual cylinder length=0.17650000000000002 radius=0.0076
- added link wamv/front_right_camera_link, mass 0.3; collision box size=0.036 0.03 0.03; collision cylinder length=0.042 radius=0.015
- added link wamv/front_right_camera_link_optical
- added link wamv/front_right_camera_post_arm_link, mass 0.1; collision cylinder length=0.065 radius=0.008; visual mesh filename=package://vrx_gazebo/models/sensor_post/mesh/sensor_post_ar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
- added link wamv/front_right_camera_post_link, mass 0.15885000000000002; collision cylinder length=0.17650000000000002 radius=0.0076; visual cylinder length=0.17650000000000002 radius=0.0076
- added link wamv/lidar_wamv_link, mass 1; collision cylinder length=0.075 radius=0.055; visual mesh filename=package://vrx_gazebo/models/3d_lidar/mesh/3d_lidar.dae
- added link wamv/lidar_wamv_post_arm_link, mass 0.1; collision cylinder length=0.065 radius=0.008; visual mesh filename=package://vrx_gazebo/models/sensor_post/mesh/sensor_post_ar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
- added link wamv/lidar_wamv_post_link, mass 0.40815000000000007; collision cylinder length=0.45350000000000007 radius=0.0076; visual cylinder length=0.45350000000000007 radius=0.0076
Joints:
- added joint wamv/base_to_far_left_camera_post_joint: type fixed, parent wamv/base_link, child wamv/far_left_camera_post_link, origin xyz=0.7 0.3 1.38475 rpy=0 0 0.0
- added joint wamv/base_to_front_left_camera_post_joint: type fixed, parent wamv/base_link, child wamv/front_left_camera_post_link, origin xyz=0.7 0.1 1.38475 rpy=0 0 0.0
- added joint wamv/base_to_front_right_camera_post_joint: type fixed, parent wamv/base_link, child wamv/front_right_camera_post_link, origin xyz=0.7 -0.1 1.38475 rpy=0 0 0.0
- added joint wamv/base_to_lidar_wamv_post_joint: type fixed, parent wamv/base_link, child wamv/lidar_wamv_post_link, origin xyz=0.6299999999999999 0.0 1.52325 rpy=0 0 0.0
- added joint wamv/far_left_camera_post_arm_to_far_left_camera_joint: type fixed, parent wamv/far_left_camera_post_arm_link, child wamv/far_left_camera_link, origin xyz=0.02 0 0.027 rpy=0.0 0.2617993877991494 0.0
- added joint wamv/far_left_camera_post_to_far_left_camera_post_arm_joint: type fixed, parent wamv/far_left_camera_post_link, child wamv/far_left_camera_post_arm_link, origin xyz=0.03 0 0.08825000000000008 rpy=0 0 0
- added joint wamv/far_left_camera_to_far_left_camera_link_optical_joint: type fixed, parent wamv/far_left_camera_link, child wamv/far_left_camera_link_optical, origin xyz=0 0 0 rpy=-1.5707963267948966 0 -1.5707963267948966
- added joint wamv/front_left_camera_post_arm_to_front_left_camera_joint: type fixed, parent wamv/front_left_camera_post_arm_link, child wamv/front_left_camera_link, origin xyz=0.02 0 0.027 rpy=0.0 0.2617993877991494 0.0
- added joint wamv/front_left_camera_post_to_front_left_camera_post_arm_joint: type fixed, parent wamv/front_left_camera_post_link, child wamv/front_left_camera_post_arm_link, origin xyz=0.03 0 0.08825000000000008 rpy=0 0 0
- added joint wamv/front_left_camera_to_front_left_camera_link_optical_joint: type fixed, parent wamv/front_left_camera_link, child wamv/front_left_camera_link_optical, origin xyz=0 0 0 rpy=-1.5707963267948966 0 -1.5707963267948966
- added joint wamv/front_right_camera_post_arm_to_front_right_camera_joint: type fixed, parent wamv/front_right_camera_post_arm_link, child wamv/front_right_camera_link, origin xyz=0.02 0 0.027 rpy=0.0 0.2617993877991494 0.0
- added joint wamv/front_right_camera_post_to_front_right_camera_post_arm_joint: type fixed, parent wamv/front_right_camera_post_link, child wamv/front_right_camera_post_arm_link, origin xyz=0.03 0 0.08825000000000008 rpy=0 0 0
- added joint wamv/front_right_camera_to_front_right_camera_link_optical_joint: type fixed, parent wamv/front_right_camera_link, child wamv/front_right_camera_link_optical, origin xyz=0 0 0 rpy=-1.5707963267948966 0 -1.5707963267948966
- added joint wamv/lidar_wamv_post_arm_to_lidar_wamv_joint: type fixed, parent wamv/lidar_wamv_post_arm_link, child wamv/lidar_wamv_link, origin xyz=0.04 0 0.05 rpy=0.0 0.13962634015954636 0.0
- added joint wamv/lidar_wamv_post_to_lidar_wamv_post_arm_joint: type fixed, parent wamv/lidar_wamv_post_link, child wamv/lidar_wamv_post_arm_link, origin xyz=0.03 0 0.22675000000000006 rpy=0 0 0

File: all_seaing_ros2/urdf/xdrive_wamv/xdrive_component_config.xacro (robot description, xacro)
@@ -6,4 +6,10 @@
     <!-- === wamv_gps === -->
       <xacro:wamv_gps name="gps_wamv" x="-0.65" y="0.0" z="1.3" R="0.0" P="0.0" Y="0.0" />
+    <!-- === wamv_camera === -->
+      <xacro:wamv_camera name="front_left_camera" visualize="False" x="0.75" y="0.1" z="1.5" R="0.0" P="${radians(15)}" Y="0.0" post_Y="0.0" />
+      <xacro:wamv_camera name="front_right_camera" visualize="False" x="0.75" y="-0.1" z="1.5" R="0.0" P="${radians(15)}" Y="0.0" post_Y="0.0" />
+      <xacro:wamv_camera name="far_left_camera" visualize="False" x="0.75" y="0.3" z="1.5" R="0.0" P="${radians(15)}" Y="0.0" post_Y="0.0" />
+    <!-- === lidar === -->
+      <xacro:lidar name="lidar_wamv" type="32_beam" x="0.7" y="0.0" z="1.8" R="0.0" P="${radians(8)}" Y="0.0" post_Y="0.0" />
   </xacro:macro>
 </robot>
