Commit message: changed gazebo verbosity and fixed missing frame error

File: all_seaing_description/urdf/simple_wamv/wamv_target.urdf (robot description, URDF)
Before this commit: robot WAM-V, 28 links, 27 joints
Links:
- removed link wamv/left_engine_link
- removed link wamv/left_propeller_link
- removed link wamv/right_engine_link
- removed link wamv/right_propeller_link
- added link wamv/back_left_engine_link, mass 15; collision box size=0.12 0.15 0.12; collision box size=0.2 0.15 0.83
- added link wamv/back_left_propeller_link, mass 0.5; collision cylinder length=0.18 radius=0.24; visual mesh filename=package://wamv_description/models/propeller/mesh/propeller.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
- added link wamv/back_right_engine_link, mass 15; collision box size=0.12 0.15 0.12; collision box size=0.2 0.15 0.83
- added link wamv/back_right_propeller_link, mass 0.5; collision cylinder length=0.18 radius=0.24; visual mesh filename=package://wamv_description/models/propeller/mesh/propeller.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
- added link wamv/front_left_engine_link, mass 15; collision box size=0.12 0.15 0.12; collision box size=0.2 0.15 0.83
- added link wamv/front_left_propeller_link, mass 0.5; collision cylinder length=0.18 radius=0.24; visual mesh filename=package://wamv_description/models/propeller/mesh/propeller.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
- added link wamv/front_right_engine_link, mass 15; collision box size=0.12 0.15 0.12; collision box size=0.2 0.15 0.83
- added link wamv/front_right_propeller_link, mass 0.5; collision cylinder length=0.18 radius=0.24; visual mesh filename=package://wamv_description/models/propeller/mesh/propeller.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
Joints:
- removed joint wamv/left_chassis_engine_joint
- removed joint wamv/left_engine_propeller_joint
- removed joint wamv/right_chassis_engine_joint
- removed joint wamv/right_engine_propeller_joint
- added joint wamv/back_left_chassis_engine_joint: type revolute, parent wamv/base_link, child wamv/back_left_engine_link, origin xyz=-2.4 1 0 rpy=0.0 0.0 0.7854, axis 0 0 1, limit lower=-3.141592653589793 upper=3.141592653589793 effort=10 velocity=10
- added joint wamv/back_left_engine_propeller_joint: type continuous, parent wamv/back_left_engine_link, child wamv/back_left_propeller_link, origin xyz=-0.278156 0 -0.509371 rpy=0 0 0, axis 1 0 0, limit effort=100 velocity=100
- added joint wamv/back_right_chassis_engine_joint: type revolute, parent wamv/base_link, child wamv/back_right_engine_link, origin xyz=-2.4 -1 0 rpy=0.0 0.0 -0.7854, axis 0 0 1, limit lower=-3.141592653589793 upper=3.141592653589793 effort=10 velocity=10
- added joint wamv/back_right_engine_propeller_joint: type continuous, parent wamv/back_right_engine_link, child wamv/back_right_propeller_link, origin xyz=-0.278156 0 -0.509371 rpy=0 0 0, axis 1 0 0, limit effort=100 velocity=100
- added joint wamv/front_left_chassis_engine_joint: type revolute, parent wamv/base_link, child wamv/front_left_engine_link, origin xyz=1.1 1 0 rpy=0.0 0.0 -0.7854, axis 0 0 1, limit lower=-3.141592653589793 upper=3.141592653589793 effort=10 velocity=10
- added joint wamv/front_left_engine_propeller_joint: type continuous, parent wamv/front_left_engine_link, child wamv/front_left_propeller_link, origin xyz=-0.278156 0 -0.509371 rpy=0 0 0, axis 1 0 0, limit effort=100 velocity=100
- added joint wamv/front_right_chassis_engine_joint: type revolute, parent wamv/base_link, child wamv/front_right_engine_link, origin xyz=1.1 -1 0 rpy=0.0 0.0 0.7854, axis 0 0 1, limit lower=-3.141592653589793 upper=3.141592653589793 effort=10 velocity=10
- added joint wamv/front_right_engine_propeller_joint: type continuous, parent wamv/front_right_engine_link, child wamv/front_right_propeller_link, origin xyz=-0.278156 0 -0.509371 rpy=0 0 0, axis 1 0 0, limit effort=100 velocity=100
