Commit message: changed gazebo verbosity and fixed missing frame error

File: all_seaing_description/urdf/xdrive_wamv/wamv_target.urdf (robot description, URDF)
Before this commit: robot WAM-V, 29 links, 28 joints
Links:
- added link wamv/ball_shooter_base_link, mass 0.5; visual mesh filename=package://vrx_gazebo/models/ball_shooter/meshes/ball_shoote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
- added link wamv/ball_shooter_launcher_link, mass 0.5; collision box size=0.3 0.3 0.2; visual mesh filename=package://vrx_gazebo/models/ball_shooter/meshes/ball_shoote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
- added link wamv/receiver, mass 0.1; visual sphere radius=0.01
Joints:
- added joint wamv/ball_shooter_base_joint: type revolute, parent wamv/base_link, child wamv/ball_shooter_base_link, origin xyz=0.55 -0.3 1.3 rpy=0 0 0.0, axis 0 0 1, limit lower=0.0 upper=0 effort=1000.0 velocity=0
- added joint wamv/ball_shooter_launcher_joint: type revolute, parent wamv/ball_shooter_base_link, child wamv/ball_shooter_launcher_link, origin xyz=-0.0204 0 0.107877 rpy=0 -0.3490658503988659 0, axis 0 0 1, limit lower=0.0 upper=0 effort=1000.0 velocity=0
- added joint wamv/receiver_pinger_joint: type revolute, parent wamv/base_link, child wamv/receiver, origin xyz=0 0 0 rpy=0 0 0, axis 0 0 1, limit lower=0.0 upper=0 effort=1000.0 velocity=0
- joint wamv/gps_wamv_joint: origin xyz=-0.65 0.0 1.3 rpy=0.0 0.0 0.0 -> xyz=-0.85 0.0 1.3 rpy=0.0 0.0 0.0
- joint wamv/imu_wamv_joint: origin xyz=-0.65 0.0 1.3 rpy=0.0 0.0 0.0 -> xyz=0.3 -0.2 1.3 rpy=0.0 0.0 0.0

File: all_seaing_description/urdf/xdrive_wamv/xdrive_component_config.xacro (robot description, xacro)
@@ -2,14 +2,18 @@
 <robot xmlns:xacro="http://ros.org/wiki/xacro" name="wam-v-components">
   <xacro:macro name="yaml_components">
-    <!-- === wamv_imu === -->
-      <xacro:wamv_imu name="imu_wamv" x="-0.65" y="0.0" z="1.3" R="0.0" P="0.0" Y="0.0" />
-    <!-- === wamv_gps === -->
-      <xacro:wamv_gps name="gps_wamv" x="-0.65" y="0.0" z="1.3" R="0.0" P="0.0" Y="0.0" />
     <!-- === wamv_camera === -->
       <xacro:wamv_camera name="front_left_camera" visualize="False" x="0.75" y="0.1" z="1.5" R="0.0" P="${radians(15)}" Y="0.0" post_Y="0.0" />
       <xacro:wamv_camera name="front_right_camera" visualize="False" x="0.75" y="-0.1" z="1.5" R="0.0" P="${radians(15)}" Y="0.0" post_Y="0.0" />
       <xacro:wamv_camera name="far_left_camera" visualize="False" x="0.75" y="0.3" z="1.5" R="0.0" P="${radians(15)}" Y="0.0" post_Y="0.0" />
+    <!-- === wamv_gps === -->
+      <xacro:wamv_gps name="gps_wamv" x="-0.85" y="0.0" z="1.3" R="0.0" P="0.0" Y="0.0" />
+    <!-- === wamv_imu === -->
+      <xacro:wamv_imu name="imu_wamv" x="0.3" y="-0.2" z="1.3" R="0.0" P="0.0" Y="0.0" />
     <!-- === lidar === -->
-      <xacro:lidar name="lidar_wamv" type="32_beam" x="0.7" y="0.0" z="1.8" R="0.0" P="${radians(8)}" Y="0.0" post_Y="0.0" />
+      <xacro:lidar name="lidar_wamv" type="16_beam" x="0.7" y="0.0" z="1.8" R="0.0" P="${radians(8)}" Y="0.0" post_Y="0.0" />
+    <!-- === wamv_ball_shooter === -->
+      <xacro:wamv_ball_shooter name="ball_shooter" x="0.55" y="-0.3" z="1.3" pitch="${radians(-20)}" yaw="0.0" />
+    <!-- === wamv_pinger === -->
+      <xacro:wamv_pinger sensor_name="receiver" position="1.0 0 -1.0" />
   </xacro:macro>
 </robot>

Commit message: changed to 32beam lidar

File: all_seaing_description/urdf/xdrive_wamv/wamv_target.urdf (robot description, URDF)
Before this commit: robot WAM-V, 29 links, 28 joints
Links:
- added link wamv/ball_shooter_base_link, mass 0.5; visual mesh filename=package://vrx_gazebo/models/ball_shooter/meshes/ball_shoote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
- added link wamv/ball_shooter_launcher_link, mass 0.5; collision box size=0.3 0.3 0.2; visual mesh filename=package://vrx_gazebo/models/ball_shooter/meshes/ball_shoote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
- added link wamv/receiver, mass 0.1; visual sphere radius=0.01
Joints:
- added joint wamv/ball_shooter_base_joint: type revolute, parent wamv/base_link, child wamv/ball_shooter_base_link, origin xyz=0.55 -0.3 1.3 rpy=0 0 0.0, axis 0 0 1, limit lower=0.0 upper=0 effort=1000.0 velocity=0
- added joint wamv/ball_shooter_launcher_joint: type revolute, parent wamv/ball_shooter_base_link, child wamv/ball_shooter_launcher_link, origin xyz=-0.0204 0 0.107877 rpy=0 -0.3490658503988659 0, axis 0 0 1, limit lower=0.0 upper=0 effort=1000.0 velocity=0
- added joint wamv/receiver_pinger_joint: type revolute, parent wamv/base_link, child wamv/receiver, origin xyz=0 0 0 rpy=0 0 0, axis 0 0 1, limit lower=0.0 upper=0 effort=1000.0 velocity=0
- joint wamv/gps_wamv_joint: origin xyz=-0.65 0.0 1.3 rpy=0.0 0.0 0.0 -> xyz=-0.85 0.0 1.3 rpy=0.0 0.0 0.0
- joint wamv/imu_wamv_joint: origin xyz=-0.65 0.0 1.3 rpy=0.0 0.0 0.0 -> xyz=0.3 -0.2 1.3 rpy=0.0 0.0 0.0
