Commit message: multi camera launch and config

File: all_seaing_description/urdf/fish_and_chips/sensor_mast.urdf.xacro (robot description, xacro)
@@ -4,9 +4,13 @@
     <link name="gps_link"></link>
     <link name="imu_link"></link>
-    <link name="zed_camera_link"></link>
-    <joint name="base_to_zed" type="fixed">
+    <!-- <link name="zed_camera_link"></link> -->
+    <link name="velodyne"></link>
+    <link name="zed_left_camera_optical_frame"></link>
+    <link name="back_left_oak_rgb_camera_optical_frame"></link>
+    <link name="back_right_oak_rgb_camera_optical_frame"></link>
+    <joint name="base_to_velodyne" type="fixed">
         <origin xyz="0.0 0.0 0.0" rpy="0 0 0"/>
         <parent link="base_link"/>
-        <child link="zed_camera_link"/>
+        <child link="velodyne"/>
     </joint>
     <joint name="base_to_gps" type="fixed">
@@ -20,3 +24,18 @@
         <child link="imu_link"/>
     </joint>
+    <joint name="velodyne_to_zed" type="fixed">
+        <origin xyz="0.07018073566954665 -0.10612744990375929 0.01631157058161572" rpy="1.6003576138834124 0.014907826408101659 -0.0010636379178425852"/>
+        <parent link="velodyne"/>
+        <child link="zed_left_camera_optical_frame"/>
+    </joint>
+    <joint name="velodyne_to_back_left_oak" type="fixed">
+        <origin xyz="0.07018073566954665 -0.10612744990375929 0.01631157058161572" rpy="1.6003576138834124 0.014907826408101659 -0.0010636379178425852"/>
+        <parent link="velodyne"/>
+        <child link="back_left_oak_rgb_camera_optical_frame"/>
+    </joint>
+    <joint name="velodyne_to_back_right_oak" type="fixed">
+        <origin xyz="0.07018073566954665 -0.10612744990375929 0.01631157058161572" rpy="1.6003576138834124 0.014907826408101659 -0.0010636379178425852"/>
+        <parent link="velodyne"/>
+        <child link="back_right_oak_rgb_camera_optical_frame"/>
+    </joint>
 </robot>

Commit message: 3-camera setup

File: all_seaing_description/urdf/fish_and_chips/sensor_mast.urdf.xacro (robot description, xacro)
@@ -25,15 +25,15 @@
     </joint>
     <joint name="velodyne_to_zed" type="fixed">
-        <origin xyz="0.07018073566954665 -0.10612744990375929 0.01631157058161572" rpy="1.6003576138834124 0.014907826408101659 -0.0010636379178425852"/>
+        <origin xyz="0.08630218352284266 0.12692593166077154 -0.3" rpy="-1.57079632679 0.0 0.04528359010351771"/>
         <parent link="velodyne"/>
         <child link="zed_left_camera_optical_frame"/>
     </joint>
     <joint name="velodyne_to_back_left_oak" type="fixed">
-        <origin xyz="0.07018073566954665 -0.10612744990375929 0.01631157058161572" rpy="1.6003576138834124 0.014907826408101659 -0.0010636379178425852"/>
+        <origin xyz="-0.05 0.12692593166077154 -0.3" rpy="-1.57079632679 0.0 2.1515106255173375"/>
         <parent link="velodyne"/>
         <child link="back_left_oak_rgb_camera_optical_frame"/>
     </joint>
     <joint name="velodyne_to_back_right_oak" type="fixed">
-        <origin xyz="0.07018073566954665 -0.10612744990375929 0.01631157058161572" rpy="1.6003576138834124 0.014907826408101659 -0.0010636379178425852"/>
+        <origin xyz="-0.05 -0.12692593166077154 -0.3" rpy="-1.57079632679 0.0 -1.8155163505207363"/>
         <parent link="velodyne"/>
         <child link="back_right_oak_rgb_camera_optical_frame"/>

Commit message: multicamera works, tuned calibration and matching weights and clusters are really good now

File: all_seaing_description/urdf/fish_and_chips/sensor_mast.urdf.xacro (robot description, xacro)
@@ -25,15 +25,15 @@
     </joint>
     <joint name="velodyne_to_zed" type="fixed">
-        <origin xyz="0.08630218352284266 0.12692593166077154 -0.3" rpy="-1.57079632679 0.0 0.04528359010351771"/>
+        <origin xyz="0.08630218352284266 0.12692593166077154 -0.27" rpy="-1.6 0.0 0.12"/>
         <parent link="velodyne"/>
         <child link="zed_left_camera_optical_frame"/>
     </joint>
     <joint name="velodyne_to_back_left_oak" type="fixed">
-        <origin xyz="-0.05 0.12692593166077154 -0.3" rpy="-1.57079632679 0.0 2.1515106255173375"/>
+        <origin xyz="-0.05 0.12692593166077154 -0.25" rpy="-1.53 0.0 1.87"/>
         <parent link="velodyne"/>
         <child link="back_left_oak_rgb_camera_optical_frame"/>
     </joint>
     <joint name="velodyne_to_back_right_oak" type="fixed">
-        <origin xyz="-0.05 -0.12692593166077154 -0.3" rpy="-1.57079632679 0.0 -1.8155163505207363"/>
+        <origin xyz="-0.05 -0.12692593166077154 -0.25" rpy="-1.57079632679 0.0 -1.80"/>
         <parent link="velodyne"/>
         <child link="back_right_oak_rgb_camera_optical_frame"/>

Commit message: slam with 3 camera system setup, outdoors testing to be done

File: all_seaing_description/urdf/fish_and_chips/sensor_mast.urdf.xacro (robot description, xacro)
@@ -10,5 +10,5 @@
     <link name="back_right_oak_rgb_camera_optical_frame"></link>
     <joint name="base_to_velodyne" type="fixed">
-        <origin xyz="0.0 0.0 0.0" rpy="0 0 0"/>
+        <origin xyz="0.0 0.0 0.0" rpy="0 0 -${pi/2}"/>
         <parent link="base_link"/>
         <child link="velodyne"/>

Commit message: Update sensor_mast.urdf.xacro
remove debug code

File: all_seaing_description/urdf/fish_and_chips/sensor_mast.urdf.xacro (robot description, xacro)
@@ -4,5 +4,4 @@
     <link name="gps_link"></link>
     <link name="imu_link"></link>
-    <!-- <link name="zed_camera_link"></link> -->
     <link name="velodyne"></link>
     <link name="zed_left_camera_optical_frame"></link>

Commit message: GPS translation from base_link reflected in URDF

File: all_seaing_description/urdf/fish_and_chips/sensor_mast.urdf.xacro (robot description, xacro)
@@ -14,5 +14,5 @@
     </joint>
     <joint name="base_to_gps" type="fixed">
-        <origin xyz="0.0 0.0 0.0" rpy="0 0 0"/>
+        <origin xyz="20.0 0.0 0.0" rpy="0 0 0"/>
         <parent link="base_link"/>
         <child link="gps_link"/>

Commit message: recalibrated for testing, will now need to recalibrate again bc of reprinted sensor mast

File: all_seaing_description/urdf/fish_and_chips/sensor_mast.urdf.xacro (robot description, xacro)
@@ -24,15 +24,15 @@
     </joint>
     <joint name="velodyne_to_zed" type="fixed">
-        <origin xyz="0.08630218352284266 0.12692593166077154 -0.27" rpy="-1.6 0.0 0.12"/>
+        <origin xyz="0.08630218352284266 0.12692593166077154 -0.27" rpy="-1.6 0.0 0.035"/>
         <parent link="velodyne"/>
         <child link="zed_left_camera_optical_frame"/>
     </joint>
     <joint name="velodyne_to_back_left_oak" type="fixed">
-        <origin xyz="-0.05 0.12692593166077154 -0.25" rpy="-1.53 0.0 1.87"/>
+        <origin xyz="-0.05 0.12692593166077154 -0.25" rpy="-1.53 0.0 1.815"/>
         <parent link="velodyne"/>
         <child link="back_left_oak_rgb_camera_optical_frame"/>
     </joint>
     <joint name="velodyne_to_back_right_oak" type="fixed">
-        <origin xyz="-0.05 -0.12692593166077154 -0.25" rpy="-1.57079632679 0.0 -1.80"/>
+        <origin xyz="-0.05 -0.12692593166077154 -0.25" rpy="-1.57079632679 0.0 -1.85"/>
         <parent link="velodyne"/>
         <child link="back_right_oak_rgb_camera_optical_frame"/>

Commit message: recalibrating and some slam changes

File: all_seaing_description/urdf/fish_and_chips/sensor_mast.urdf.xacro (robot description, xacro)
@@ -19,20 +19,20 @@
     </joint>
     <joint name="base_to_imu" type="fixed">
-        <origin xyz="0.0 0.0 0.0" rpy="0 0 ${pi/2}"/>
+        <origin xyz="0.0 0.0 0.0" rpy="0 0 -${pi/2}"/>
         <parent link="base_link"/>
         <child link="imu_link"/>
     </joint>
     <joint name="velodyne_to_zed" type="fixed">
-        <origin xyz="0.08630218352284266 0.12692593166077154 -0.27" rpy="-1.6 0.0 0.035"/>
+        <origin xyz="0.08630218352284266 0.12692593166077154 -0.27" rpy="-1.6 0.0 0.012"/>
         <parent link="velodyne"/>
         <child link="zed_left_camera_optical_frame"/>
     </joint>
     <joint name="velodyne_to_back_left_oak" type="fixed">
-        <origin xyz="-0.05 0.12692593166077154 -0.25" rpy="-1.53 0.0 1.815"/>
+        <origin xyz="-0.05 0.12692593166077154 -0.25" rpy="-1.57079632679 0.0 1.905"/>
         <parent link="velodyne"/>
         <child link="back_left_oak_rgb_camera_optical_frame"/>
     </joint>
     <joint name="velodyne_to_back_right_oak" type="fixed">
-        <origin xyz="-0.05 -0.12692593166077154 -0.25" rpy="-1.57079632679 0.0 -1.85"/>
+        <origin xyz="-0.05 -0.12692593166077154 -0.25" rpy="-1.57079632679 0.0 -1.795"/>
         <parent link="velodyne"/>
         <child link="back_right_oak_rgb_camera_optical_frame"/>

Commit message: IMU-GPS fusion working now, aligned IMU frame to have correct odometry twist direction, attempted fusing internal Pixhawk EKF with IMU & GPS data in the localization node but having frame issues (odometry is misaligned)

File: all_seaing_description/urdf/fish_and_chips/sensor_mast.urdf.xacro (robot description, xacro)
@@ -4,4 +4,5 @@
     <link name="gps_link"></link>
     <link name="imu_link"></link>
+    <link name="imu_link_fake"></link>
     <link name="velodyne"></link>
     <link name="zed_left_camera_optical_frame"></link>
@@ -9,5 +10,5 @@
     <link name="back_right_oak_rgb_camera_optical_frame"></link>
     <joint name="base_to_velodyne" type="fixed">
-        <origin xyz="0.0 0.0 0.0" rpy="0 0 -${pi/2}"/>
+        <origin xyz="0.0 0.0 0.0" rpy="0 0 0"/>
         <parent link="base_link"/>
         <child link="velodyne"/>
@@ -19,7 +20,12 @@
     </joint>
     <joint name="base_to_imu" type="fixed">
-        <origin xyz="0.0 0.0 0.0" rpy="0 0 -${pi/2}"/>
+        <origin xyz="0.0 0.0 0.0" rpy="0 ${pi} -${pi/2}"/>
         <parent link="base_link"/>
         <child link="imu_link"/>
+    </joint>
+    <joint name="base_to_imu_fake" type="fixed">
+        <origin xyz="0.0 0.0 0.0" rpy="0 ${pi} ${pi/2}"/>
+        <parent link="base_link"/>
+        <child link="imu_link_fake"/>
     </joint>
     <joint name="velodyne_to_zed" type="fixed">

Commit message: localization (roughly, just not that bad) working with internal Pixhawk EKF, SLAM fine-tuning (there is a bug but predicted location and map is pretty stable)

File: all_seaing_description/urdf/fish_and_chips/sensor_mast.urdf.xacro (robot description, xacro)
@@ -3,6 +3,6 @@
     <link name="base_link"></link>
     <link name="gps_link"></link>
-    <link name="imu_link"></link>
-    <link name="imu_link_fake"></link>
+    <link name="imu_link_accel"></link>
+    <link name="imu_link_odom"></link>
     <link name="velodyne"></link>
     <link name="zed_left_camera_optical_frame"></link>
@@ -10,5 +10,5 @@
     <link name="back_right_oak_rgb_camera_optical_frame"></link>
     <joint name="base_to_velodyne" type="fixed">
-        <origin xyz="0.0 0.0 0.0" rpy="0 0 0"/>
+        <origin xyz="0.0 0.0 0.0" rpy="0 0 -${pi/2}"/>
         <parent link="base_link"/>
         <child link="velodyne"/>
@@ -19,26 +19,26 @@
         <child link="gps_link"/>
     </joint>
-    <joint name="base_to_imu" type="fixed">
-        <origin xyz="0.0 0.0 0.0" rpy="0 ${pi} -${pi/2}"/>
+    <joint name="base_to_imu_accel" type="fixed">
+        <origin xyz="0.0 0.0 0.0" rpy="0 0 ${pi/2}"/>
         <parent link="base_link"/>
-        <child link="imu_link"/>
+        <child link="imu_link_accel"/>
     </joint>
-    <joint name="base_to_imu_fake" type="fixed">
-        <origin xyz="0.0 0.0 0.0" rpy="0 ${pi} ${pi/2}"/>
+    <joint name="base_to_imu_odom" type="fixed">
+        <origin xyz="0.0 0.0 0.0" rpy="0 0 -${pi/2}"/>
         <parent link="base_link"/>
-        <child link="imu_link_fake"/>
+        <child link="imu_link_odom"/>
     </joint>
     <joint name="velodyne_to_zed" type="fixed">
-        <origin xyz="0.08630218352284266 0.12692593166077154 -0.27" rpy="-1.6 0.0 0.012"/>
+        <origin xyz="-0.12692593166077154 0.08630218352284266 -0.27" rpy="-1.6 0.0 0.012"/>
         <parent link="velodyne"/>
         <child link="zed_left_camera_optical_frame"/>
     </joint>
     <joint name="velodyne_to_back_left_oak" type="fixed">
-        <origin xyz="-0.05 0.12692593166077154 -0.25" rpy="-1.57079632679 0.0 1.905"/>
+        <origin xyz="-0.12692593166077154 -0.05 -0.25" rpy="-1.57079632679 0.0 1.905"/>
         <parent link="velodyne"/>
         <child link="back_left_oak_rgb_camera_optical_frame"/>
     </joint>
     <joint name="velodyne_to_back_right_oak" type="fixed">
-        <origin xyz="-0.05 -0.12692593166077154 -0.25" rpy="-1.57079632679 0.0 -1.795"/>
+        <origin xyz="0.12692593166077154 -0.05 -0.25" rpy="-1.57079632679 0.0 -1.795"/>
         <parent link="velodyne"/>
         <child link="back_right_oak_rgb_camera_optical_frame"/>

Commit message: fix perception on roboboat rosbag (lidar cluster pre-filtering doesn't work long-range, clusters too small), LIO setup, utm in locations

File: all_seaing_description/urdf/fish_and_chips/sensor_mast.urdf.xacro (robot description, xacro)
@@ -20,5 +20,5 @@
     </joint>
     <joint name="base_to_imu_accel" type="fixed">
-        <origin xyz="0.0 0.0 0.0" rpy="0 0 ${pi/2}"/>
+        <origin xyz="0.0 0.0 0.0" rpy="0 0 -${pi/2}"/>
         <parent link="base_link"/>
         <child link="imu_link_accel"/>

Commit message: correct acceleration frame (upside down + flip gyro) & removing gravity

File: all_seaing_description/urdf/fish_and_chips/sensor_mast.urdf.xacro (robot description, xacro)
@@ -19,13 +19,13 @@
         <child link="gps_link"/>
     </joint>
-    <joint name="base_to_imu_accel" type="fixed">
-        <origin xyz="0.0 0.0 0.0" rpy="0 0 -${pi/2}"/>
-        <parent link="base_link"/>
-        <child link="imu_link_accel"/>
-    </joint>
     <joint name="base_to_imu_odom" type="fixed">
         <origin xyz="0.0 0.0 0.0" rpy="0 0 -${pi/2}"/>
         <parent link="base_link"/>
         <child link="imu_link_odom"/>
+    </joint>
+    <joint name="imu_odom_to_imu_accel" type="fixed">
+        <origin xyz="0.0 0.0 0.0" rpy="${pi} 0 0"/>
+        <parent link="imu_link_odom"/>
+        <child link="imu_link_accel"/>
     </joint>
     <joint name="velodyne_to_zed" type="fixed">

Commit message: changed calibration based on cad of new sensor mast

File: all_seaing_description/urdf/fish_and_chips/sensor_mast.urdf.xacro (robot description, xacro)
@@ -30,15 +30,15 @@
     </joint>
     <joint name="velodyne_to_zed" type="fixed">
-        <origin xyz="-0.12692593166077154 0.08630218352284266 -0.27" rpy="-1.6 0.0 0.012"/>
+        <origin xyz="-0.06 0.11237 -0.27" rpy="-1.6 0.0 0.0"/>
         <parent link="velodyne"/>
         <child link="zed_left_camera_optical_frame"/>
     </joint>
     <joint name="velodyne_to_back_left_oak" type="fixed">
-        <origin xyz="-0.12692593166077154 -0.05 -0.25" rpy="-1.57079632679 0.0 1.905"/>
+        <origin xyz="-0.07 -0.023 -0.25" rpy="-1.57079632679 0.0 1.87623"/>
         <parent link="velodyne"/>
         <child link="back_left_oak_rgb_camera_optical_frame"/>
     </joint>
     <joint name="velodyne_to_back_right_oak" type="fixed">
-        <origin xyz="0.12692593166077154 -0.05 -0.25" rpy="-1.57079632679 0.0 -1.795"/>
+        <origin xyz="0.07 -0.023 -0.25" rpy="-1.57079632679 0.0 -1.87623"/>
         <parent link="velodyne"/>
         <child link="back_right_oak_rgb_camera_optical_frame"/>

Commit message: test changes

File: all_seaing_description/urdf/fish_and_chips/sensor_mast.urdf.xacro (robot description, xacro)
@@ -35,10 +35,10 @@
     </joint>
     <joint name="velodyne_to_back_left_oak" type="fixed">
-        <origin xyz="-0.07 -0.023 -0.25" rpy="-1.57079632679 0.0 1.87623"/>
+        <origin xyz="-0.118 0.008 -0.24" rpy="-1.57079632679 0.0 1.01259265359"/>
         <parent link="velodyne"/>
         <child link="back_left_oak_rgb_camera_optical_frame"/>
     </joint>
     <joint name="velodyne_to_back_right_oak" type="fixed">
-        <origin xyz="0.07 -0.023 -0.25" rpy="-1.57079632679 0.0 -1.87623"/>
+        <origin xyz="0.118 0.008 -0.24" rpy="-1.57079632679 0.0 -1.01259265359"/>
         <parent link="velodyne"/>
         <child link="back_right_oak_rgb_camera_optical_frame"/>

Commit message: new sensor mast

File: all_seaing_description/urdf/fish_and_chips/sensor_mast.urdf.xacro (robot description, xacro)
@@ -30,15 +30,15 @@
     </joint>
     <joint name="velodyne_to_zed" type="fixed">
-        <origin xyz="-0.06 0.11237 -0.27" rpy="-1.6 0.0 0.0"/>
+        <origin xyz="-0.06 0.11237 -0.175" rpy="-1.6 0.0 0.0"/>
         <parent link="velodyne"/>
         <child link="zed_left_camera_optical_frame"/>
     </joint>
     <joint name="velodyne_to_back_left_oak" type="fixed">
-        <origin xyz="-0.118 0.008 -0.24" rpy="-1.57079632679 0.0 1.01259265359"/>
+        <origin xyz="-0.118 0.008 -0.145" rpy="-1.57079632679 0.0 1.01259265359"/>
         <parent link="velodyne"/>
         <child link="back_left_oak_rgb_camera_optical_frame"/>
     </joint>
     <joint name="velodyne_to_back_right_oak" type="fixed">
-        <origin xyz="0.118 0.008 -0.24" rpy="-1.57079632679 0.0 -1.01259265359"/>
+        <origin xyz="0.118 0.008 -0.145" rpy="-1.57079632679 0.0 -1.01259265359"/>
         <parent link="velodyne"/>
         <child link="back_right_oak_rgb_camera_optical_frame"/>

Commit message: test changes

File: all_seaing_description/urdf/fish_and_chips/sensor_mast.urdf.xacro (robot description, xacro)
@@ -30,15 +30,15 @@
     </joint>
     <joint name="velodyne_to_zed" type="fixed">
-        <origin xyz="-0.06 0.11237 -0.175" rpy="-1.6 0.0 0.0"/>
+        <origin xyz="-0.06 0.11237 -0.10" rpy="-1.6 0.0 0.0"/>
         <parent link="velodyne"/>
         <child link="zed_left_camera_optical_frame"/>
     </joint>
     <joint name="velodyne_to_back_left_oak" type="fixed">
-        <origin xyz="-0.118 0.008 -0.145" rpy="-1.57079632679 0.0 1.01259265359"/>
+        <origin xyz="-0.118 0.008 -0.07" rpy="-1.57079632679 0.0 1.01259265359"/>
         <parent link="velodyne"/>
         <child link="back_left_oak_rgb_camera_optical_frame"/>
     </joint>
     <joint name="velodyne_to_back_right_oak" type="fixed">
-        <origin xyz="0.118 0.008 -0.145" rpy="-1.57079632679 0.0 -1.01259265359"/>
+        <origin xyz="0.118 0.008 -0.07" rpy="-1.57079632679 0.0 -1.01259265359"/>
         <parent link="velodyne"/>
         <child link="back_right_oak_rgb_camera_optical_frame"/>

Commit message: im stupid

File: all_seaing_description/urdf/fish_and_chips/sensor_mast.urdf.xacro (robot description, xacro)
@@ -15,5 +15,5 @@
     </joint>
     <joint name="base_to_gps" type="fixed">
-        <origin xyz="20.0 0.0 0.0" rpy="0 0 0"/>
+        <origin xyz="0.2 0.0 0.0" rpy="0 0 0"/>
         <parent link="base_link"/>
         <child link="gps_link"/>
